Commit message: Temp commit, non function code

File: p5_ws/src/lbr_fri/lbr_fri_ros2_stack/lbr_ros2_control/config/lbr_system_interface.xacro (robot description, xacro)
@@ -2,16 +2,21 @@
 <robot xmlns:xacro="http://www.ros.org/wiki/xacro">
     <xacro:macro name="lbr_system_interface"
-        params="sim joint_limits system_parameters_path">
+        params="mode joint_limits system_parameters_path">
         <!-- load system parameters via yaml -->
         <xacro:property name="system_parameters"
             value="${xacro.load_yaml(system_parameters_path)}" />
         <ros2_control name="lbr_system_interface" type="system">
-            <!-- define hardware including parameters, also gazebo -->
-            <xacro:if value="${sim}">
+            <!-- load plugin depending on mode -->
+            <xacro:if value="${mode == 'mock'}">
                 <hardware>
-                    <plugin>gazebo_ros2_control/GazeboSystem</plugin>
+                    <plugin>mock_components/GenericSystem</plugin>
                 </hardware>
             </xacro:if>
-            <xacro:unless value="${sim}">
+            <xacro:if value="${mode == 'gazebo'}">
+                <hardware>
+                    <plugin>ign_ros2_control/IgnitionSystem</plugin>
+                </hardware>
+            </xacro:if>
+            <xacro:if value="${mode == 'hardware'}">
                 <hardware>
                     <plugin>lbr_ros2_control::SystemInterface</plugin>
@@ -33,8 +38,8 @@
                     <param name="open_loop">${system_parameters['hardware']['open_loop']}</param>
                 </hardware>
-            </xacro:unless>
+            </xacro:if>
             <!-- define lbr specific state interfaces as sensor, see
             https://github.com/ros-controls/roadmap/blob/master/design_drafts/components_architecture_and_urdf_examples.md -->
-            <xacro:unless value="${sim}">
+            <xacro:if value="${mode == 'hardware'}">
                 <sensor name="auxiliary_sensor">
                     <!-- see KUKA::FRI::LBRState -->
@@ -80,25 +85,29 @@
                     <command_interface name="torque.z" />
                 </gpio>
-            </xacro:unless>
+            </xacro:if>
             <!-- define joints and command/state interfaces for each joint -->
             <xacro:macro name="joint_interface"
-                params="name min_position max_position max_velocity max_torque sim">
+                params="name min_position max_position max_velocity max_torque mode">
                 <joint name="${name}">
-                    <param name="min_position">${min_position}</param>
-                    <param name="max_position">${max_position}</param>
-                    <param name="max_velocity">${max_velocity}</param>
-                    <param name="max_torque">${max_torque}</param>
                     <command_interface name="position">
                         <param name="min">${min_position}</param>
                         <param name="max">${max_position}</param>
                     </command_interface>
-                    <command_interface name="effort">
-                        <param name="min">-${max_torque}</param>
-                        <param name="max"> ${max_torque}</param>
-                    </command_interface>
+                    <!-- only single command interface, refer
+                    https://github.com/ros-controls/gz_ros2_control/issues/182 -->
+                    <xacro:unless value="${mode == 'gazebo'}">
+                        <command_interface name="effort">
+                            <param name="min">-${max_torque}</param>
+                            <param name="max"> ${max_torque}</param>
+                        </command_interface>
+                    </xacro:unless>
                     <state_interface name="position" />
                     <state_interface name="velocity" />
                     <state_interface name="effort" />
-                    <xacro:unless value="${sim}">
+                    <xacro:if value="${mode == 'hardware'}">
+                        <param name="min_position">${min_position}</param>
+                        <param name="max_position">${max_position}</param>
+                        <param name="max_velocity">${max_velocity}</param>
+                        <param name="max_torque">${max_torque}</param>
                         <xacro:if value="${system_parameters['hardware']['fri_client_sdk']['major_version'] == 1}">
                             <state_interface name="commanded_joint_position" />
@@ -107,5 +116,5 @@
                         <state_interface name="external_torque" />
                         <state_interface name="ipo_joint_position" />
-                    </xacro:unless>
+                    </xacro:if>
                 </joint>
             </xacro:macro>
@@ -115,5 +124,5 @@
                 max_velocity="${joint_limits['A1']['velocity'] * PI / 180}"
                 max_torque="${joint_limits['A1']['effort']}"
-                sim="${sim}" />
+                mode="${mode}" />
             <xacro:joint_interface name="A2"
                 min_position="${joint_limits['A2']['lower'] * PI / 180}"
@@ -121,5 +130,5 @@
                 max_velocity="${joint_limits['A2']['velocity'] * PI / 180}"
                 max_torque="${joint_limits['A2']['effort']}"
-                sim="${sim}" />
+                mode="${mode}" />
             <xacro:joint_interface name="A3"
                 min_position="${joint_limits['A3']['lower'] * PI / 180}"
@@ -127,5 +136,5 @@
                 max_velocity="${joint_limits['A3']['velocity'] * PI / 180}"
                 max_torque="${joint_limits['A3']['effort']}"
-                sim="${sim}" />
+                mode="${mode}" />
             <xacro:joint_interface name="A4"
                 min_position="${joint_limits['A4']['lower'] * PI / 180}"
@@ -133,5 +142,5 @@
                 max_velocity="${joint_limits['A4']['velocity'] * PI / 180}"
                 max_torque="${joint_limits['A4']['effort']}"
-                sim="${sim}" />
+                mode="${mode}" />
             <xacro:joint_interface name="A5"
                 min_position="${joint_limits['A5']['lower'] * PI / 180}"
@@ -139,5 +148,5 @@
                 max_velocity="${joint_limits['A5']['velocity'] * PI / 180}"
                 max_torque="${joint_limits['A5']['effort']}"
-                sim="${sim}" />
+                mode="${mode}" />
             <xacro:joint_interface name="A6"
                 min_position="${joint_limits['A6']['lower'] * PI / 180}"
@@ -145,5 +154,5 @@
                 max_velocity="${joint_limits['A6']['velocity'] * PI / 180}"
                 max_torque="${joint_limits['A6']['effort']}"
-                sim="${sim}" />
+                mode="${mode}" />
             <xacro:joint_interface name="A7"
                 min_position="${joint_limits['A7']['lower'] * PI / 180}"
@@ -151,5 +160,5 @@
                 max_velocity="${joint_limits['A7']['velocity'] * PI / 180}"
                 max_torque="${joint_limits['A7']['effort']}"
-                sim="${sim}" />
+                mode="${mode}" />
         </ros2_control>
     </xacro:macro>

File: p5_ws/src/robutler/kuka_table_description/urdf/iiwa7_table_xacro/iiwa7.xacro (robot description, xacro)
@@ -9,26 +9,29 @@
         name="system_parameters_path"
         default="$(find lbr_ros2_control)/config/lbr_system_parameters.yaml" />
+    <material name="steel_satin">
+        <color rgba="0.6274509803921569 0.6274509803921569 0.6274509803921569 1.0"/>
+    </material>
     <!-- fixed to world, see http://classic.gazebosim.org/tutorials?tut=ros_urdf&cat=connect_ros -->
     <link name="world" />
-     <!-- Table link -->
+    <!-- table mount -->
     <link name="table">
-      <inertial>
-        <origin rpy="0 0 0" xyz="0.47511520643410643 0.9340356249199337 1.753635248949686"/>
-        <mass value="1382.7919279449686"/>
-        <inertia ixx="1994.27355" ixy="-0.365832" ixz="-0.552572" iyy="2787.103818" iyz="-145.275916" izz="966.579181"/>
-      </inertial>
-      <visual>
-        <origin rpy="0 0 0" xyz="0 0 0"/>
-        <geometry>
-          <mesh filename="package://kuka_bord_description/meshes/table_meshes/visual/base_link.stl" scale="0.001 0.001 0.001"/>
-        </geometry>
-        <material name="steel_satin"/>
-      </visual>
-      <collision>
-        <origin rpy="0 0 0" xyz="0 0 0"/>
-        <geometry>
-          <mesh filename="package://kuka_bord_description/meshes/table_meshes/collision/base_link_low_polly.stl" scale="0.001 0.001 0.001"/>
-        </geometry>
-      </collision>
+        <inertial>
+            <origin xyz="0.47511520643410643 0.9340356249199337 1.753635248949686" rpy="0 0 0"/>
+            <mass value="1382.7919279449686"/>
+            <inertia ixx="1994.27355" iyy="2787.103818" izz="966.579181" ixy="-0.365832" iyz="-145.275916" ixz="-0.552572"/>
+        </inertial>
+        <visual>
+            <origin xyz="0 0 0" rpy="0 0 0"/>
+            <geometry>
+                <mesh filename="package://kuka_table_description/meshes/table_meshes/visual/base_link.stl" scale="0.001 0.001 0.001"/>
+            </geometry>
+            <material name="steel_satin"/>
+        </visual>
+        <collision>
+            <origin xyz="0 0 0" rpy="0 0 0"/>
+            <geometry>
+                <mesh filename="package://kuka_table_description/meshes/table_meshes/collision/base_link_low_polly.stl" scale="0.001 0.001 0.001"/>
+            </geometry>
+        </collision>
     </link>
     <!--joint between world and table-->
@@ -37,10 +40,11 @@
         <child link="table" />
     </joint>
-    <!-- joint between table and iiwa7-->
-    <joint name="world_joint" type="fixed">
+    <!--joint between table and right iiwa7 -->
+    <joint name="mount_right" type="fixed">
         <parent link="table" />
         <child link="link_0" />
         <origin xyz="0.273705 0.76 1.037203" rpy="0.785398163 0 -1.57079633"/>
     </joint>
+    <!--<origin xyz="0.716295 0.76 1.037203" rpy="-0.785398163 0 -1.57079633"/>-->
     <!-- iiwa -->
     <xacro:iiwa7

File: p5_ws/src/robutler/kuka_table_description/urdf/iiwa7_table_xacro/iiwa7_description.xacro (robot description, xacro)
@@ -3,5 +3,5 @@
     <!-- robot as extracted via https://github.com/syuntoku14/fusion2urdf -->
     <xacro:macro name="iiwa7"
-        params="robot_name:=^|lbr mode:= mock system_parameters_path:=^|'$(find lbr_ros2_control)/config/lbr_system_parameters.yaml'">
+        params="robot_name:=^|lbr mode:=^|mock system_parameters_path:=^|'$(find lbr_ros2_control)/config/lbr_system_parameters.yaml'">
         <!-- includes -->
         <xacro:include filename="$(find lbr_description)/gazebo/lbr_gazebo.xacro" />
