Commit message: Updated gripper and fixed set_moveit_coords depend

File: p5_ws/src/lbr_fri/lbr_fri_ros2_stack/lbr_description/urdf/iiwa7_table_new/iiwa7_table.xacro (robot description, xacro)
@@ -16,5 +16,5 @@
     </material>
     <material name="wood">
-        <color rgba="0.6274509803921569 0.6274509803921569 0.6274509803921569 1.0"/>
+        <color rgba="0.588235294 0.375 0 1.0"/>
     </material>
     <!-- fixed to world, see http://classic.gazebosim.org/tutorials?tut=ros_urdf&cat=connect_ros -->
@@ -42,15 +42,20 @@
     </link>
     <link name="cam_mount">
+        <inertial>
+            <origin xyz="0.47511520643410643 0.9340356249199337 1.753635248949686" rpy="0 0 0"/>
+            <mass value="1382.7919279449686"/>
+            <inertia ixx="1994.27355" iyy="2787.103818" izz="966.579181" ixy="-0.365832" iyz="-145.275916" ixz="-0.552572"/>
+        </inertial>
         <visual>
             <origin xyz="-0.096012 -0.03490 59.336" rpy="0 0 0"/>
             <geometry>
-                <mesh filename="package://lbr_description/meshes/table/visual/base_link.stl" scale="0.001 0.001 0.001"/>
+                <mesh filename="package://lbr_description/meshes/camera_mount/Camera_Mount_V2_v2.stl" scale="0.001 0.001 0.001"/>
             </geometry>
-            <material name="steel_satin"/>
+            <material name="wood"/>
         </visual>
         <collision>
-            <origin xyz="0 0 0" rpy="0 0 0"/>
+            <origin xyz="-0.096012 -0.03490 59.336" rpy="0 0 0"/>
             <geometry>
-                <mesh filename="package://lbr_description/meshes/table/collision/base_link_low_polly.stl" scale="0.001 0.001 0.001"/>
+                <mesh filename="package://lbr_description/meshes/camera_mount/Camera_Mount_V2_v2.stl" scale="0.001 0.001 0.001"/>
             </geometry>
         </collision>
@@ -60,4 +65,10 @@
         <parent link="world" />
         <child link="table" />
+    </joint>
+    <!--joint between table and camera mount-->
+    <joint name="cam_table_joint" type="fixed">
+        <parent link="table" />
+        <child link="cam_mount" />
+        <origin xyz="0.489819 0.84691 1.428" rpy="0 0 0"/>
     </joint>
     <!--joint between table and right iiwa7 -->

File: p5_ws/src/lbr_fri/lbr_fri_ros2_stack/lbr_description/urdf/robotiq-3f-gripper/robotiq-3f-gripper_finger_articulated_macro.xacro (robot description, xacro)
@@ -21,5 +21,5 @@
 				<origin xyz="0.020 0 0" rpy="0 0 0"/>
 				<geometry>
-                                        <mesh filename="package://lbr_description/meshes/robotiq-3f-gripper_articulated/collision/link_0.stl" />
+                                        <mesh filename="package://lbr_description/meshes/robotiq-3f-gripper_articulated/collision/link_0.STL" />
 				</geometry>
 				<material name="yellow">
@@ -44,5 +44,5 @@
 				<origin xyz="0.050 -.028 0" rpy="0 0 -0.52"/>
 				<geometry>
-                                        <mesh filename="package://lbr_description/meshes/robotiq-3f-gripper_articulated/collision/link_1.stl" />
+                                        <mesh filename="package://lbr_description/meshes/robotiq-3f-gripper_articulated/collision/link_1.STL" />
 				</geometry>
 				<material name="yellow"/>
@@ -65,5 +65,5 @@
 				<origin xyz="0.039 0 0.0075" rpy="0 0 0"/>
 				<geometry>
-                                        <mesh filename="package://lbr_description/meshes/robotiq-3f-gripper_articulated/collision/link_2.stl" />
+                                        <mesh filename="package://lbr_description/meshes/robotiq-3f-gripper_articulated/collision/link_2.STL" />
 				</geometry>
 				<material name="yellow"/>
@@ -86,5 +86,5 @@
 				<origin xyz="0 0 0" rpy="0 0 0.52"/>
 				<geometry>
-                                        <mesh filename="package://lbr_description/meshes/robotiq-3f-gripper_articulated/collision/link_3.stl" />
+                                        <mesh filename="package://lbr_description/meshes/robotiq-3f-gripper_articulated/collision/link_3.STL" />
 				</geometry>
 				<material name="yellow"/>
