Commit message: Updated kinematic solver and endefector

File: p5_ws/src/lbr_fri/lbr_fri_ros2_stack/lbr_description/urdf/iiwa7_table_cali/iiwa7_table_cali.xacro (robot description, xacro)
@@ -2,17 +2,15 @@
 <!-- top level -->
 <robot name="iiwa7_table" xmlns:xacro="http://www.ros.org/wiki/xacro">
-    <!-- include the lbr iiwa7 macro -->
-    <xacro:include filename="$(find lbr_description)/urdf/iiwa7_table/iiwa7_table_description.xacro" />
-    <!-- include 3f gripper and set its macro prefix to 3f-->
+    <!-- include the lbr iiwa macro -->
+    <xacro:include filename="$(find lbr_description)/urdf/iiwa7_table_cali/iiwa7_table_cali_description.xacro" />
+    <!-- include 3f gripper and set its macro prefix to 3f-
     <xacro:include filename="$(find lbr_description)/urdf/robotiq-3f-gripper/robotiq-3f-gripper_articulated_macro.xacro" />
     <xacro:robotiq-3f-gripper_articulated prefix="3f_" />
-    <!-- include realsense camera -->
-    <xacro:include filename="$(find lbr_description)/urdf/realsense/_d435.urdf.xacro" />
+    -->
     <xacro:arg name="robot_name" default="lbr" />
-    <xacro:arg name="sim" default="false" />
+    <xacro:arg name="sim" default="true" />
     <xacro:arg
         name="system_parameters_path"
         default="$(find lbr_ros2_control)/config/lbr_system_parameters.yaml" />
-    <!-- materials -->
     <material name="steel_satin">
         <color rgba="0.6274509803921569 0.6274509803921569 0.6274509803921569 1"/>
@@ -26,5 +24,5 @@
     <!-- fixed to world, see http://classic.gazebosim.org/tutorials?tut=ros_urdf&cat=connect_ros -->
     <link name="world" />
-    <!-- table link -->
+    <!-- table mount -->
     <link name="table">
         <inertial>
@@ -47,5 +45,4 @@
         </collision>
     </link>
-    <!-- the wooden laser cut camera mount-->
     <link name="cam_mount">
         <visual>
@@ -56,4 +53,20 @@
             <material name="wood"/>
         </visual>
+        <!-- Might want to add collision, tho the table takes care of it-->
+    </link>
+    <link name="tip">
+        <visual>
+            <origin xyz="0 0 0" rpy="0 0 0"/>
+            <geometry>
+                <mesh filename="package://lbr_description/meshes/calibration_tip/calli_tip.stl" scale="0.001 0.001 0.001"/>
+            </geometry>
+            <material name="white"/>
+        </visual>
+        <collision>
+            <origin xyz="0 0 0" rpy="0 0 0"/>
+            <geometry>
+                <mesh filename="package://lbr_description/meshes/calibration_tip/calli_tip.stl" scale="0.001 0.001 0.001"/>
+            </geometry>
+        </collision>
     </link>
     <!--joint between world and table-->
@@ -62,5 +75,5 @@
         <child link="table" />
     </joint>
-    <!--joint between table and wooden camera mount-->
+    <!--joint between table and camera mount-->
     <joint name="cam_table_joint" type="fixed">
         <parent link="table" />
@@ -77,10 +90,14 @@
     <joint name="ee_mount" type="fixed">
         <parent link="link_ee" />
-        <child link="3f_palm" />
-        <origin xyz="0 0 0.05" rpy="1.57079633 0 0"/>
+        <child link="tip" />
+        <origin xyz="0 0 0" rpy="0 0 0"/>
     </joint>
-    <!-- joint between wooden camera mount and camera, done using d435 xacro macro
-    <xacro:sensor_d435 parent="table" name="camera" origin="xyz='0 0 0.1' rpy='0 0 0'" />
-    -->
+    <!-- joint between 3d-printed tip and it's tip-->
+    <link name = "tip_point" />
+    <joint name="tip_point" type="fixed">
+        <parent link="tip" />
+        <child link="tip_point" />
+        <origin xyz="0 0 0.05" rpy="0 0 0"/>
+    </joint>
     <!-- Left iiwa7 (Needs to be uptated) <origin xyz="0.716295 0.76 1.037203" rpy="-0.785398163 0 -1.57079633"/>-->
     <!-- iiwa -->
@@ -89,3 +106,3 @@
         sim="$(arg sim)"
         system_parameters_path="$(arg system_parameters_path)" />
-    </robot>
+</robot>

File: p5_ws/src/lbr_fri/lbr_fri_ros2_stack/lbr_description/urdf/iiwa7_table_cali/iiwa7_table_cali_description.xacro (robot description, xacro)
@@ -1,4 +1,3 @@
 <?xml version="1.0"?>
-<!-- the right iiwa7 -->
 <robot xmlns:xacro="http://www.ros.org/wiki/xacro">
     <!-- robot as extracted via https://github.com/syuntoku14/fusion2urdf -->

File: p5_ws/src/lbr_fri/lbr_fri_ros2_stack/lbr_description/urdf/realsense/_d435.urdf.xacro (robot description, xacro)
@@ -21,7 +21,7 @@
 <robot name="sensor_d435" xmlns:xacro="http://ros.org/wiki/xacro">
   <!-- Includes -->
-  <xacro:include filename="$(find lbr_description)/urdf/left_arm/_materials.urdf.xacro" />
-  <xacro:include filename="$(find lbr_description)/urdf/left_arm/_usb_plug.urdf.xacro" />
-  <xacro:macro name="sensor_d435" params="parent *origin name:=camera use_nominal_extrinsics:=false add_plug:=false use_mesh:=true">
+  <xacro:include filename="$(find lbr_description)/urdf/realsense/_materials.urdf.xacro" />
+  <xacro:include filename="$(find lbr_description)/urdf/realsense/_usb_plug.urdf.xacro" />
+  <xacro:macro name="sensor_d435" params="parent origin name:=camera use_nominal_extrinsics:=false add_plug:=false use_mesh:=true">
     <xacro:property name="M_PI" value="3.1415926535897931" />
     <!-- The following values are approximate, and the camera node
@@ -42,5 +42,5 @@
     <xacro:property name="d435_zero_depth_to_glass" value="4.2e-3"/>
     <!-- convenience precomputation to avoid clutter-->
-    <xacro:property name="d435_mesh_x_offset" value="${d435_cam_mount_from_center_offset-d435_glass_to_front-d435_zero_depth_to_glass}"/>
+    <xacro:property name="d435_mesh_x_offset" value="${d435_cam_mount_f rom_center_offset-d435_glass_to_front-d435_zero_depth_to_glass}"/>
     <!-- The following offset is relative the the physical D435 camera peripherial
   	camera tripod mount -->

Commit message: Moved the point around which the arm moves, so it is positioned at the tip of the gripper fingers

File: p5_ws/src/lbr_fri/lbr_fri_ros2_stack/lbr_description/urdf/iiwa7_table_cali/iiwa7_table_cali.xacro (robot description, xacro)
@@ -53,5 +53,5 @@
             <material name="wood"/>
         </visual>
-        <!-- Might want to add collision, tho the table takes care of it-->
+        <!-- no need for collision, this is added in the table collision-->
     </link>
     <link name="tip">

File: p5_ws/src/lbr_fri/lbr_fri_ros2_stack/lbr_description/urdf/robotiq-3f-gripper/robotiq-3f-gripper_articulated_macro.xacro (robot description, xacro)
@@ -63,5 +63,5 @@
 			<parent link="${prefix}palm"/>
 			<child link="${prefix}tool0"/>
-			<origin xyz="0.0 0.0875 0.0" rpy="0 0 1.5707"/>
+			<origin xyz="0.0 0.18 0" rpy="0 0 1.5707"/>
 		</joint>
 		<!-- end of joint list -->
