Commit message: New low polly collision stl for faster loading time

File: p5_ws/src/lbr_fri/lbr_fri_ros2_stack/lbr_description/urdf/iiwa7_table/iiwa7_table.xacro (robot description, xacro)
@@ -24,5 +24,5 @@
             <origin xyz="0 0 0" rpy="0 0 0"/>
             <geometry>
-                <mesh filename="package://lbr_description/meshes/table/visual/base_link.stl" scale="0.001 0.001 0.001"/>
+                <mesh filename="package://lbr_description/meshes/table/visual/base_link_low_polly.stl" scale="0.001 0.001 0.001"/>
             </geometry>
             <material name="steel_satin"/>
@@ -31,5 +31,5 @@
             <origin xyz="0 0 0" rpy="0 0 0"/>
             <geometry>
-                <mesh filename="package://lbr_description/meshes/table/collision/base_link_low_polly.stl" scale="0.001 0.001 0.001"/>
+                <mesh filename="package://lbr_description/meshes/table/collision/iiwa7_table_collision.stl" scale="0.001 0.001 0.001"/>
             </geometry>
         </collision>

File: p5_ws/src/lbr_fri/lbr_fri_ros2_stack/lbr_description/urdf/iiwa7_table_new/iiwa7_table.xacro (robot description, xacro)
@@ -13,8 +13,11 @@
         default="$(find lbr_ros2_control)/config/lbr_system_parameters.yaml" />
     <material name="steel_satin">
-        <color rgba="0.6274509803921569 0.6274509803921569 0.6274509803921569 1.0"/>
+        <color rgba="0.6274509803921569 0.6274509803921569 0.6274509803921569 1"/>
     </material>
     <material name="wood">
-        <color rgba="0.588235294 0.375 0 1.0"/>
+        <color rgba="0.588235294 0.375 0.1 1"/>
+    </material>
+    <material name="red">
+        <color rgba="1 0 0 1"/>
     </material>
     <!-- fixed to world, see http://classic.gazebosim.org/tutorials?tut=ros_urdf&cat=connect_ros -->
@@ -30,5 +33,5 @@
             <origin xyz="0 0 0" rpy="0 0 0"/>
             <geometry>
-                <mesh filename="package://lbr_description/meshes/table/visual/base_link.stl" scale="0.001 0.001 0.001"/>
+                <mesh filename="package://lbr_description/meshes/table/visual/base_link_low_polly.stl" scale="0.001 0.001 0.001"/>
             </geometry>
             <material name="steel_satin"/>
@@ -37,16 +40,11 @@
             <origin xyz="0 0 0" rpy="0 0 0"/>
             <geometry>
-                <mesh filename="package://lbr_description/meshes/table/collision/base_link_low_polly.stl" scale="0.001 0.001 0.001"/>
+                <mesh filename="package://lbr_description/meshes/table/collision/iiwa7_table_collision.stl" scale="0.001 0.001 0.001"/>
             </geometry>
         </collision>
     </link>
     <link name="cam_mount">
-        <inertial>
-            <origin xyz="0.47511520643410643 0.9340356249199337 1.753635248949686" rpy="0 0 0"/>
-            <mass value="1382.7919279449686"/>
-            <inertia ixx="1994.27355" iyy="2787.103818" izz="966.579181" ixy="-0.365832" iyz="-145.275916" ixz="-0.552572"/>
-        </inertial>
         <visual>
-            <origin xyz="-0.096012 -0.03490 59.336" rpy="0 0 0"/>
+            <origin xyz="0.096012 0.03490 -0.59336" rpy="0 0 0"/>
             <geometry>
                 <mesh filename="package://lbr_description/meshes/camera_mount/Camera_Mount_V2_v2.stl" scale="0.001 0.001 0.001"/>
@@ -55,5 +53,5 @@
         </visual>
         <collision>
-            <origin xyz="-0.096012 -0.03490 59.336" rpy="0 0 0"/>
+            <origin xyz="0.096012 0.03490 -0.59336" rpy="0 0 0"/>
             <geometry>
                 <mesh filename="package://lbr_description/meshes/camera_mount/Camera_Mount_V2_v2.stl" scale="0.001 0.001 0.001"/>

Commit message: Added gripper to the moveit config

File: p5_ws/src/lbr_fri/lbr_fri_ros2_stack/lbr_description/urdf/iiwa7_table/iiwa7_table.xacro (robot description, xacro)
@@ -4,4 +4,7 @@
     <!-- include the lbr iiwa macro -->
     <xacro:include filename="$(find lbr_description)/urdf/iiwa7_table/iiwa7_table_description.xacro" />
+    <!-- include 3f gripper and set its macro prefix to 3f-->
+    <xacro:include filename="$(find lbr_description)/urdf/robotiq-3f-gripper/robotiq-3f-gripper_articulated_macro.xacro" />
+    <xacro:robotiq-3f-gripper_articulated prefix="3f_" />
     <xacro:arg name="robot_name" default="lbr" />
     <xacro:arg name="sim" default="true" />
@@ -10,5 +13,11 @@
         default="$(find lbr_ros2_control)/config/lbr_system_parameters.yaml" />
     <material name="steel_satin">
-        <color rgba="0.6274509803921569 0.6274509803921569 0.6274509803921569 1.0"/>
+        <color rgba="0.6274509803921569 0.6274509803921569 0.6274509803921569 1"/>
+    </material>
+    <material name="wood">
+        <color rgba="0.588235294 0.375 0.1 1"/>
+    </material>
+    <material name="red">
+        <color rgba="1 0 0 1"/>
     </material>
     <!-- fixed to world, see http://classic.gazebosim.org/tutorials?tut=ros_urdf&cat=connect_ros -->
@@ -35,4 +44,19 @@
         </collision>
     </link>
+    <link name="cam_mount">
+        <visual>
+            <origin xyz="0.096012 0.03490 -0.059336" rpy="0 0 0"/>
+            <geometry>
+                <mesh filename="package://lbr_description/meshes/camera_mount/Camera_Mount_V2_v2.stl" scale="0.001 0.001 0.001"/>
+            </geometry>
+            <material name="wood"/>
+        </visual>
+        <collision>
+            <origin xyz="0.096012 0.03490 -0.059336" rpy="0 0 0"/>
+            <geometry>
+                <mesh filename="package://lbr_description/meshes/camera_mount/Camera_Mount_V2_v2.stl" scale="0.001 0.001 0.001"/>
+            </geometry>
+        </collision>
+    </link>
     <!--joint between world and table-->
     <joint name="world_joint" type="fixed">
@@ -40,11 +64,23 @@
         <child link="table" />
     </joint>
+    <!--joint between table and camera mount-->
+    <joint name="cam_table_joint" type="fixed">
+        <parent link="table" />
+        <child link="cam_mount" />
+        <origin xyz="0.489819 0.84691 1.428" rpy="1.57079633 0 0"/>
+    </joint>
     <!--joint between table and right iiwa7 -->
     <joint name="mount_right" type="fixed">
         <parent link="table" />
         <child link="link_0" />
-        <origin xyz="0.273705 0.76 1.037203" rpy="0.785398163 0 -1.57079633"/>
+        <origin xyz="0.268524 0.756691 1.037203" rpy="0.785398163 0 -1.57079633"/>
     </joint>
-    <!--<origin xyz="0.716295 0.76 1.037203" rpy="-0.785398163 0 -1.57079633"/>-->
+    <!-- joint between right iiwa7 and 3f gripper-->
+    <joint name="ee_mount" type="fixed">
+        <parent link="link_ee" />
+        <child link="3f_palm" />
+        <origin xyz="0 0 0.05" rpy="1.57079633 0 0"/>
+    </joint>
+    <!-- Left iiwa7 (Needs to be uptated) <origin xyz="0.716295 0.76 1.037203" rpy="-0.785398163 0 -1.57079633"/>-->
     <!-- iiwa -->
     <xacro:iiwa7_table

Commit message: Added gripper mounting plate STL file and implemented it in iiwa7_table.xacro

File: p5_ws/src/lbr_fri/lbr_fri_ros2_stack/lbr_description/urdf/iiwa7_table/iiwa7_table.xacro (robot description, xacro)
@@ -57,4 +57,19 @@
         </visual>
     </link>
+    <link name="gripper_mounting_plate">
+        <visual>
+            <origin xyz="0.045 0.045 0" rpy="0 0 0"/>
+            <geometry>
+                <mesh filename="package://lbr_description/meshes/gripper_mounting_plate/gripper_mounting_plate.stl" scale="0.001 0.001 0.001"/>
+            </geometry>
+            <material name="steel_satin"/>
+        </visual>
+        <collision>
+            <origin xyz="0.045 0.045 0" rpy="0 0 0"/>
+            <geometry>
+                <mesh filename="package://lbr_description/meshes/gripper_mounting_plate/gripper_mounting_plate.stl" scale="0.001 0.001 0.001"/>
+            </geometry>
+        </collision>
+    </link>
     <!--joint between world and table-->
     <joint name="world_joint" type="fixed">
@@ -77,4 +92,10 @@
     <joint name="ee_mount" type="fixed">
         <parent link="link_ee" />
+        <child link="gripper_mounting_plate" />
+        <origin xyz="0 0 0.05" rpy="1.57079633 0 0"/>
+    </joint>
+    <!-- joint between right iiwa7 and 3f gripper-->
+    <joint name="adapter_mount" type="fixed">
+        <parent link="gripper_mounting_plate" />
         <child link="3f_palm" />
         <origin xyz="0 0 0.05" rpy="1.57079633 0 0"/>

Commit message: Updated xacro and SRDF with gripper adapter plate

File: p5_ws/src/lbr_fri/lbr_fri_ros2_stack/lbr_description/urdf/iiwa7_table/iiwa7_table.xacro (robot description, xacro)
@@ -59,5 +59,5 @@
     <link name="gripper_mounting_plate">
         <visual>
-            <origin xyz="0.045 0.045 0" rpy="0 0 0"/>
+            <origin xyz="0.045 -0.045 0" rpy="0 0 0"/>
             <geometry>
                 <mesh filename="package://lbr_description/meshes/gripper_mounting_plate/gripper_mounting_plate.stl" scale="0.001 0.001 0.001"/>
@@ -66,5 +66,5 @@
         </visual>
         <collision>
-            <origin xyz="0.045 0.045 0" rpy="0 0 0"/>
+            <origin xyz="0.045 -0.045 0" rpy="0 0 0"/>
             <geometry>
                 <mesh filename="package://lbr_description/meshes/gripper_mounting_plate/gripper_mounting_plate.stl" scale="0.001 0.001 0.001"/>
@@ -93,5 +93,5 @@
         <parent link="link_ee" />
         <child link="gripper_mounting_plate" />
-        <origin xyz="0 0 0.05" rpy="1.57079633 0 0"/>
+        <origin xyz="0 0 0" rpy="0 0 0"/>
     </joint>
     <!-- joint between right iiwa7 and 3f gripper-->
@@ -99,5 +99,5 @@
         <parent link="gripper_mounting_plate" />
         <child link="3f_palm" />
-        <origin xyz="0 0 0.05" rpy="1.57079633 0 0"/>
+        <origin xyz="0 0 0.0745" rpy="1.57079633 0 0"/>
     </joint>
     <!-- joint between wooden camera mount and camera, done using d435 xacro macro
