Commit message: temp

File: p5_ws/src/lbr_fri/lbr_fri_ros2_stack/lbr_description/urdf/robotiq-3f-gripper/robotiq-3f-gripper_articulated_macro.xacro (robot description, xacro)
@@ -63,5 +63,5 @@
 			<parent link="${prefix}palm"/>
 			<child link="${prefix}tool0"/>
-			<origin xyz="0.0 0.18 0" rpy="0 0 1.5707"/>
+			<origin xyz="0.0 0.18 0" rpy="0 0 -1.5707"/>
 		</joint>
 		<!-- end of joint list -->

Commit message: Calibrated the transformation matrices

File: p5_ws/src/lbr_fri/lbr_fri_ros2_stack/lbr_description/urdf/robotiq-3f-gripper/robotiq-3f-gripper_articulated_macro.xacro (robot description, xacro)
@@ -63,5 +63,5 @@
 			<parent link="${prefix}palm"/>
 			<child link="${prefix}tool0"/>
-			<origin xyz="0.0 0.18 0" rpy="0 0 1.5707"/>
+			<origin xyz="0.0 0.18 0" rpy="0 -1.5707 1.5707"/>
 		</joint>
 		<!-- end of joint list -->

Commit message: Updated planner, so now the parameters in OMPL_planning.yaml acutally are loaded, instead of the default

File: p5_ws/src/lbr_fri/lbr_fri_ros2_stack/lbr_description/urdf/robotiq-3f-gripper/robotiq-3f-gripper_articulated_macro.xacro (robot description, xacro)
@@ -63,5 +63,5 @@
 			<parent link="${prefix}palm"/>
 			<child link="${prefix}tool0"/>
-			<origin xyz="0.0 0.18 0" rpy="0 0 -1.5707"/>
+			<origin xyz="0.0 0.18 0" rpy="0 1.5707 -1.5707"/>
 		</joint>
 		<!-- end of joint list -->
