Commit message: Both Robot arms - with their controllers - works with demo.launch

File: p5_ws/src/lbr_fri/lbr_fri_ros2_stack/lbr_description/urdf/dual_arm/dual_arm_w_gazebo.xacro (robot description, xacro)
@@ -1,5 +1,5 @@
 <?xml version="1.0" ?>
 <!-- =================================================================================== -->
-<!-- |    This document was autogenerated by xacro from src/lbr_fri/lbr_fri_ros2_stack/lbr_description/urdf/dual_arm/dual_arm.xacro | -->
+<!-- |    This document was autogenerated by xacro from dual_arm_refreshed.xacro       | -->
 <!-- |    EDITING THIS FILE BY HAND IS NOT RECOMMENDED                                 | -->
 <!-- =================================================================================== -->
@@ -9,65 +9,76 @@
     <xacro:include filename="$(find lbr_description)/urdf/dual_arm/dual_arm_description.xacro" />
     -->
+  <!-- ros_control-plugin -->
+  <gazebo>
+    <plugin filename="libgazebo_ros2_control.so" name="gazebo_ros2_control">
+      <parameters>/home/thor/P5-Kuka-Dual-Arm/p5_ws/install/lbr_ros2_control_right/share/lbr_ros2_control_right/config/lbr_controllers_right.yaml</parameters>
+      <ros>
+        <namespace>/lbr</namespace>
+        <!-- remapping for controller manager inside Gazebo plugin -->
+        <remapping>~/robot_description:=robot_description</remapping>
+      </ros>
+    </plugin>
+  </gazebo>
+  <gazebo reference="right_link_0">
+    <mu1>0.2</mu1>
+    <mu2>0.2</mu2>
+  </gazebo>
+  <gazebo reference="right_A1">
+    <implicitSpringDamper>true</implicitSpringDamper>
+    <provideFeedback>true</provideFeedback>
+  </gazebo>
+  <gazebo reference="right_link_1">
+    <mu1>0.2</mu1>
+    <mu2>0.2</mu2>
+  </gazebo>
+  <gazebo reference="right_A2">
+    <implicitSpringDamper>true</implicitSpringDamper>
+    <provideFeedback>true</provideFeedback>
+  </gazebo>
+  <gazebo reference="right_link_2">
+    <mu1>0.2</mu1>
+    <mu2>0.2</mu2>
+  </gazebo>
+  <gazebo reference="right_A3">
+    <implicitSpringDamper>true</implicitSpringDamper>
+    <provideFeedback>true</provideFeedback>
+  </gazebo>
+  <gazebo reference="right_link_3">
+    <mu1>0.2</mu1>
+    <mu2>0.2</mu2>
+  </gazebo>
+  <gazebo reference="right_A4">
+    <implicitSpringDamper>true</implicitSpringDamper>
+    <provideFeedback>true</provideFeedback>
+  </gazebo>
+  <gazebo reference="right_link_4">
+    <mu1>0.2</mu1>
+    <mu2>0.2</mu2>
+  </gazebo>
+  <gazebo reference="right_A5">
+    <implicitSpringDamper>true</implicitSpringDamper>
+    <provideFeedback>true</provideFeedback>
+  </gazebo>
+  <gazebo reference="right_link_5">
+    <mu1>0.2</mu1>
+    <mu2>0.2</mu2>
+  </gazebo>
+  <gazebo reference="right_A6">
+    <implicitSpringDamper>true</implicitSpringDamper>
+    <provideFeedback>true</provideFeedback>
+  </gazebo>
+  <gazebo reference="right_link_6">
+    <mu1>0.2</mu1>
+    <mu2>0.2</mu2>
+  </gazebo>
+  <gazebo reference="right_A7">
+    <implicitSpringDamper>true</implicitSpringDamper>
+    <provideFeedback>true</provideFeedback>
+  </gazebo>
+  <gazebo reference="right_link_7">
+    <mu1>0.2</mu1>
+    <mu2>0.2</mu2>
+  </gazebo>
   <ros2_control name="lbr_system_interface_right" type="system">
-    <hardware>
-      <plugin>lbr_ros2_control::SystemInterface</plugin>
-      <param name="fri_client_sdk_major_version">1</param>
-      <param name="fri_client_sdk_minor_version">15</param>
-      <param name="client_command_mode">position</param>
-      <param name="port_id">30200</param>
-      <param name="remote_host">INADDR_ANY</param>
-      <param name="rt_prio">80</param>
-      <param name="pid_p">0.1</param>
-      <param name="pid_i">0.0</param>
-      <param name="pid_d">0.0</param>
-      <param name="pid_i_max">0.0</param>
-      <param name="pid_i_min">0.0</param>
-      <param name="pid_antiwindup">False</param>
-      <param name="command_guard_variant">default</param>
-      <param name="external_torque_cutoff_frequency">10</param>
-      <param name="measured_torque_cutoff_frequency">10</param>
-      <param name="open_loop">True</param>
-    </hardware>
-    <sensor name="auxiliary_sensor">
-      <!-- see KUKA::FRI::LBRState -->
-      <state_interface name="sample_time"/>
-      <state_interface name="session_state"/>
-      <state_interface name="connection_quality"/>
-      <state_interface name="safety_state"/>
-      <state_interface name="operation_mode"/>
-      <state_interface name="drive_state"/>
-      <state_interface name="client_command_mode"/>
-      <state_interface name="overlay_type"/>
-      <state_interface name="control_mode"/>
-      <state_interface name="time_stamp_sec"/>
-      <state_interface name="time_stamp_nano_sec"/>
-      <state_interface name="tracking_performance"/>
-    </sensor>
-    <sensor name="estimated_ft_sensor">
-      <param name="chain_root">right_link_0</param>
-      <param name="chain_tip">right_link_ee</param>
-      <param name="damping">0.2</param>
-      <param name="force_x_th">2.0</param>
-      <param name="force_y_th">2.0</param>
-      <param name="force_z_th">2.0</param>
-      <param name="torque_x_th">0.5</param>
-      <param name="torque_y_th">0.5</param>
-      <param name="torque_z_th">0.5</param>
-      <state_interface name="force.x"/>
-      <state_interface name="force.y"/>
-      <state_interface name="force.z"/>
-      <state_interface name="torque.x"/>
-      <state_interface name="torque.y"/>
-      <state_interface name="torque.z"/>
-    </sensor>
-    <!-- FRI Cartesian impedance control mode -->
-    <gpio name="wrench">
-      <command_interface name="force.x"/>
-      <command_interface name="force.y"/>
-      <command_interface name="force.z"/>
-      <command_interface name="torque.x"/>
-      <command_interface name="torque.y"/>
-      <command_interface name="torque.z"/>
-    </gpio>
     <joint name="right_A1">
       <param name="min_position">-2.9670597283903604</param>
@@ -86,8 +97,4 @@
       <state_interface name="velocity"/>
       <state_interface name="effort"/>
-      <state_interface name="commanded_joint_position"/>
-      <state_interface name="commanded_torque"/>
-      <state_interface name="external_torque"/>
-      <state_interface name="ipo_joint_position"/>
     </joint>
     <joint name="right_A2">
@@ -107,8 +114,4 @@
       <state_interface name="velocity"/>
       <state_interface name="effort"/>
-      <state_interface name="commanded_joint_position"/>
-      <state_interface name="commanded_torque"/>
-      <state_interface name="external_torque"/>
-      <state_interface name="ipo_joint_position"/>
     </joint>
     <joint name="right_A3">
@@ -128,8 +131,4 @@
       <state_interface name="velocity"/>
       <state_interface name="effort"/>
-      <state_interface name="commanded_joint_position"/>
-      <state_interface name="commanded_torque"/>
-      <state_interface name="external_torque"/>
-      <state_interface name="ipo_joint_position"/>
     </joint>
     <joint name="right_A4">
@@ -149,8 +148,4 @@
       <state_interface name="velocity"/>
       <state_interface name="effort"/>
-      <state_interface name="commanded_joint_position"/>
-      <state_interface name="commanded_torque"/>
-      <state_interface name="external_torque"/>
-      <state_interface name="ipo_joint_position"/>
     </joint>
     <joint name="right_A5">
@@ -170,8 +165,4 @@
       <state_interface name="velocity"/>
       <state_interface name="effort"/>
-      <state_interface name="commanded_joint_position"/>
-      <state_interface name="commanded_torque"/>
-      <state_interface name="external_torque"/>
-      <state_interface name="ipo_joint_position"/>
     </joint>
     <joint name="right_A6">
@@ -191,8 +182,4 @@
       <state_interface name="velocity"/>
       <state_interface name="effort"/>
-      <state_interface name="commanded_joint_position"/>
-      <state_interface name="commanded_torque"/>
-      <state_interface name="external_torque"/>
-      <state_interface name="ipo_joint_position"/>
     </joint>
     <joint name="right_A7">
@@ -212,8 +199,4 @@
       <state_interface name="velocity"/>
       <state_interface name="effort"/>
-      <state_interface name="commanded_joint_position"/>
-      <state_interface name="commanded_torque"/>
-      <state_interface name="external_torque"/>
-      <state_interface name="ipo_joint_position"/>
     </joint>
   </ros2_control>
@@ -433,65 +416,76 @@
   <link name="right_link_ee">
         </link>
+  <!-- ros_control-plugin -->
+  <gazebo>
+    <plugin filename="libgazebo_ros2_control.so" name="gazebo_ros2_control">
+      <parameters>/home/thor/P5-Kuka-Dual-Arm/p5_ws/install/lbr_ros2_control_left/share/lbr_ros2_control_left/config/lbr_controllers_left.yaml</parameters>
+      <ros>
+        <namespace>/lbr</namespace>
+        <!-- remapping for controller manager inside Gazebo plugin -->
+        <remapping>~/robot_description:=robot_description</remapping>
+      </ros>
+    </plugin>
+  </gazebo>
+  <gazebo reference="left_link_0">
+    <mu1>0.2</mu1>
+    <mu2>0.2</mu2>
+  </gazebo>
+  <gazebo reference="left_A1">
+    <implicitSpringDamper>true</implicitSpringDamper>
+    <provideFeedback>true</provideFeedback>
+  </gazebo>
+  <gazebo reference="left_link_1">
+    <mu1>0.2</mu1>
+    <mu2>0.2</mu2>
+  </gazebo>
+  <gazebo reference="left_A2">
+    <implicitSpringDamper>true</implicitSpringDamper>
+    <provideFeedback>true</provideFeedback>
+  </gazebo>
+  <gazebo reference="left_link_2">
+    <mu1>0.2</mu1>
+    <mu2>0.2</mu2>
+  </gazebo>
+  <gazebo reference="left_A3">
+    <implicitSpringDamper>true</implicitSpringDamper>
+    <provideFeedback>true</provideFeedback>
+  </gazebo>
+  <gazebo reference="left_link_3">
+    <mu1>0.2</mu1>
+    <mu2>0.2</mu2>
+  </gazebo>
+  <gazebo reference="left_A4">
+    <implicitSpringDamper>true</implicitSpringDamper>
+    <provideFeedback>true</provideFeedback>
+  </gazebo>
+  <gazebo reference="left_link_4">
+    <mu1>0.2</mu1>
+    <mu2>0.2</mu2>
+  </gazebo>
+  <gazebo reference="left_A5">
+    <implicitSpringDamper>true</implicitSpringDamper>
+    <provideFeedback>true</provideFeedback>
+  </gazebo>
+  <gazebo reference="left_link_5">
+    <mu1>0.2</mu1>
+    <mu2>0.2</mu2>
+  </gazebo>
+  <gazebo reference="left_A6">
+    <implicitSpringDamper>true</implicitSpringDamper>
+    <provideFeedback>true</provideFeedback>
+  </gazebo>
+  <gazebo reference="left_link_6">
+    <mu1>0.2</mu1>
+    <mu2>0.2</mu2>
+  </gazebo>
+  <gazebo reference="left_A7">
+    <implicitSpringDamper>true</implicitSpringDamper>
+    <provideFeedback>true</provideFeedback>
+  </gazebo>
+  <gazebo reference="left_link_7">
+    <mu1>0.2</mu1>
+    <mu2>0.2</mu2>
+  </gazebo>
   <ros2_control name="lbr_system_interface_left" type="system">
-    <hardware>
-      <plugin>lbr_ros2_control::SystemInterface</plugin>
-      <param name="fri_client_sdk_major_version">1</param>
-      <param name="fri_client_sdk_minor_version">15</param>
-      <param name="client_command_mode">position</param>
-      <param name="port_id">30201</param>
-      <param name="remote_host">INADDR_ANY</param>
-      <param name="rt_prio">80</param>
-      <param name="pid_p">0.1</param>
-      <param name="pid_i">0.0</param>
-      <param name="pid_d">0.0</param>
-      <param name="pid_i_max">0.0</param>
-      <param name="pid_i_min">0.0</param>
-      <param name="pid_antiwindup">False</param>
-      <param name="command_guard_variant">default</param>
-      <param name="external_torque_cutoff_frequency">10</param>
-      <param name="measured_torque_cutoff_frequency">10</param>
-      <param name="open_loop">True</param>
-    </hardware>
-    <sensor name="auxiliary_sensor">
-      <!-- see KUKA::FRI::LBRState -->
-      <state_interface name="sample_time"/>
-      <state_interface name="session_state"/>
-      <state_interface name="connection_quality"/>
-      <state_interface name="safety_state"/>
-      <state_interface name="operation_mode"/>
-      <state_interface name="drive_state"/>
-      <state_interface name="client_command_mode"/>
-      <state_interface name="overlay_type"/>
-      <state_interface name="control_mode"/>
-      <state_interface name="time_stamp_sec"/>
-      <state_interface name="time_stamp_nano_sec"/>
-      <state_interface name="tracking_performance"/>
-    </sensor>
-    <sensor name="estimated_ft_sensor">
-      <param name="chain_root">left_link_0</param>
-      <param name="chain_tip">left_link_ee</param>
-      <param name="damping">0.2</param>
-      <param name="force_x_th">2.0</param>
-      <param name="force_y_th">2.0</param>
-      <param name="force_z_th">2.0</param>
-      <param name="torque_x_th">0.5</param>
-      <param name="torque_y_th">0.5</param>
-      <param name="torque_z_th">0.5</param>
-      <state_interface name="force.x"/>
-      <state_interface name="force.y"/>
-      <state_interface name="force.z"/>
-      <state_interface name="torque.x"/>
-      <state_interface name="torque.y"/>
-      <state_interface name="torque.z"/>
-    </sensor>
-    <!-- FRI Cartesian impedance control mode -->
-    <gpio name="wrench">
-      <command_interface name="force.x"/>
-      <command_interface name="force.y"/>
-      <command_interface name="force.z"/>
-      <command_interface name="torque.x"/>
-      <command_interface name="torque.y"/>
-      <command_interface name="torque.z"/>
-    </gpio>
     <joint name="left_A1">
       <param name="min_position">-2.9670597283903604</param>
@@ -510,8 +504,4 @@
       <state_interface name="velocity"/>
       <state_interface name="effort"/>
-      <state_interface name="commanded_joint_position"/>
-      <state_interface name="commanded_torque"/>
-      <state_interface name="external_torque"/>
-      <state_interface name="ipo_joint_position"/>
     </joint>
     <joint name="left_A2">
@@ -531,8 +521,4 @@
       <state_interface name="velocity"/>
       <state_interface name="effort"/>
-      <state_interface name="commanded_joint_position"/>
-      <state_interface name="commanded_torque"/>
-      <state_interface name="external_torque"/>
-      <state_interface name="ipo_joint_position"/>
     </joint>
     <joint name="left_A3">
@@ -552,8 +538,4 @@
       <state_interface name="velocity"/>
       <state_interface name="effort"/>
-      <state_interface name="commanded_joint_position"/>
-      <state_interface name="commanded_torque"/>
-      <state_interface name="external_torque"/>
-      <state_interface name="ipo_joint_position"/>
     </joint>
     <joint name="left_A4">
@@ -573,8 +555,4 @@
       <state_interface name="velocity"/>
       <state_interface name="effort"/>
-      <state_interface name="commanded_joint_position"/>
-      <state_interface name="commanded_torque"/>
-      <state_interface name="external_torque"/>
-      <state_interface name="ipo_joint_position"/>
     </joint>
     <joint name="left_A5">
@@ -594,8 +572,4 @@
       <state_interface name="velocity"/>
       <state_interface name="effort"/>
-      <state_interface name="commanded_joint_position"/>
-      <state_interface name="commanded_torque"/>
-      <state_interface name="external_torque"/>
-      <state_interface name="ipo_joint_position"/>
     </joint>
     <joint name="left_A6">
@@ -615,8 +589,4 @@
       <state_interface name="velocity"/>
       <state_interface name="effort"/>
-      <state_interface name="commanded_joint_position"/>
-      <state_interface name="commanded_torque"/>
-      <state_interface name="external_torque"/>
-      <state_interface name="ipo_joint_position"/>
     </joint>
     <joint name="left_A7">
@@ -636,8 +606,4 @@
       <state_interface name="velocity"/>
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
File: p5_ws/src/lbr_fri/lbr_fri_ros2_stack/lbr_description/urdf/iiwa7/iiwa7.xacro (robot description, xacro)
@@ -5,5 +5,5 @@
     <xacro:include filename="$(find lbr_description)/urdf/iiwa7/iiwa7_description.xacro" />
     <xacro:arg name="robot_name" default="lbr" />
-    <xacro:arg name="sim" default="true" />
+    <xacro:arg name="sim" default="false" />
     <xacro:arg
         name="system_parameters_path"

File: p5_ws/src/lbr_fri/lbr_fri_ros2_stack/lbr_description/urdf/iiwa7/iiwa7_description_macro.xacro (robot description, xacro)
@@ -16,6 +16,6 @@
         <xacro:property name="joint_friction" value="0.1" />
         <!-- parameters -->
-        <xacro:property name="system_parameters_path" value="$(find lbr_ros2_control)/config/lbr_system_parameters${suffix}.yaml"/>
-        <xacro:property name="robot_name" value="lbr${suffix}"/>
+        <xacro:property name="system_parameters_path" value="$(find lbr_ros2_control${suffix})/config/lbr_system_parameters${suffix}.yaml"/>
+        <xacro:property name="robot_name" value="lbr"/> <!--${suffix}-->
         <xacro:property name="sim" value="true"/>
         <!-- macros for simulation and real hardware -->

File: p5_ws/src/lbr_fri/lbr_fri_ros2_stack/lbr_ros2_control/config/lbr_system_interface.xacro (robot description, xacro)
@@ -7,10 +7,4 @@
             value="${xacro.load_yaml(system_parameters_path)}" />
         <ros2_control name="lbr_system_interface" type="system">
-            <!-- define hardware including parameters, also gazebo -->
-            <xacro:if value="${sim}">
-                <hardware>
-                    <plugin>gazebo_ros2_control/GazeboSystem</plugin>
-                </hardware>
-            </xacro:if>
             <xacro:unless value="${sim}">
                 <hardware>

File: p5_ws/src/lbr_fri/lbr_fri_ros2_stack/lbr_ros2_control_left/config/lbr_system_interface.xacro (robot description, xacro)
@@ -7,5 +7,4 @@
             value="${xacro.load_yaml(system_parameters_path)}" />
         <ros2_control name="lbr_system_interface" type="system">
-            <!-- define hardware including parameters, also gazebo -->
             <xacro:if value="${sim}">
                 <hardware>
