Commit message: Added 3f_gripper mounting plate, and moved left arm movepoint (2f_tool0) to right place and rotation

File: p5_ws/src/lbr_fri/lbr_fri_ros2_stack/lbr_description/urdf/dual_arm/dual_arm.xacro (robot description, xacro)
@@ -1225,4 +1225,5 @@
   </link>
   <link name="3f_tool0"/>
+  <link name="2f_tool0"/>
   <inertial>
     <origin rpy="0 0 0" xyz="0 0 0"/>
@@ -1257,5 +1258,5 @@
     <parent link="3f_palm"/>
     <child link="3f_tool0"/>
-    <origin rpy="0 -1.5707 1.5707" xyz="0.0 0.18 0"/>
+    <origin rpy="0 -1.5707 1.5707" xyz="0.0 0.17 0"/>
   </joint>
   <!-- end of joint list -->
@@ -1637,4 +1638,20 @@
     </visual>
   </link>
+  <!-- 3f gripper adapter / mounting plate -->
+  <link name="gripper_mounting_plate">
+        <visual>
+            <origin xyz="0.045 -0.045 0" rpy="0 0 0"/>
+            <geometry>
+                <mesh filename="package://lbr_description/meshes/gripper_mounting_plate/gripper_mounting_plate.stl" scale="0.001 0.001 0.001"/>
+            </geometry>
+            <material name="steel_satin"/>
+        </visual>
+        <collision>
+            <origin xyz="0.045 -0.045 0" rpy="0 0 0"/>
+            <geometry>
+                <mesh filename="package://lbr_description/meshes/gripper_mounting_plate/gripper_mounting_plate.stl" scale="0.001 0.001 0.001"/>
+            </geometry>
+        </collision>
+    </link>
   <!--joint between world and table-->
   <joint name="world_joint" type="fixed">
@@ -1655,9 +1672,15 @@
   </joint>
   <!-- joint between right iiwa7 and 3f gripper-->
-  <joint name="right_ee_mount" type="fixed">
-    <parent link="right_link_ee"/>
-    <child link="3f_palm"/>
-    <origin rpy="1.57079633 0 0" xyz="0 0 0.05"/>
-  </joint>
+    <joint name="ee_mount" type="fixed">
+        <parent link="right_link_ee" />
+        <child link="gripper_mounting_plate" />
+        <origin xyz="0 0 0" rpy="0 0 0"/>
+    </joint>
+  <!-- joint between right iiwa7 and 3f gripper-->
+    <joint name="adapter_mount" type="fixed">
+        <parent link="gripper_mounting_plate" />
+        <child link="3f_palm" />
+        <origin xyz="0 0 0.0745" rpy="1.57079633 0 -1.57079633"/>
+    </joint>
   <!-- joint between left arm and world -->
   <joint name="mount_left" type="fixed">
@@ -1672,3 +1695,9 @@
     <origin rpy="0 0 0" xyz="0 0 0"/>
   </joint>
+  <!-- joint between left arm ee and 2f gripper-->
+  <joint name="2f_ee_tool0" type="fixed">
+    <parent link="left_link_ee"/>
+    <child link="2f_tool0"/>
+    <origin rpy="0 3.14 0" xyz="0 0 0.155"/>
+  </joint>
 </robot>

Commit message: Small adjustments in xacro

File: p5_ws/src/lbr_fri/lbr_fri_ros2_stack/lbr_description/urdf/dual_arm/dual_arm.xacro (robot description, xacro)
@@ -1258,5 +1258,5 @@
     <parent link="3f_palm"/>
     <child link="3f_tool0"/>
-    <origin rpy="0 -1.5707 1.5707" xyz="0.0 0.17 0"/>
+    <origin rpy="0 -1.5707 1.5707" xyz="0.0 0.15 0"/>
   </joint>
   <!-- end of joint list -->
@@ -1699,5 +1699,5 @@
     <parent link="left_link_ee"/>
     <child link="2f_tool0"/>
-    <origin rpy="0 3.14 0" xyz="0 0 0.155"/>
+    <origin rpy="0 3.14 0" xyz="0 0 0.175"/>
   </joint>
 </robot>

Commit message: Gripper movement in moveit

File: p5_ws/src/lbr_fri/lbr_fri_ros2_stack/lbr_description/urdf/dual_arm/dual_arm.xacro (robot description, xacro)
@@ -1225,5 +1225,4 @@
   </link>
   <link name="3f_tool0"/>
-  <link name="2f_tool0"/>
   <inertial>
     <origin rpy="0 0 0" xyz="0 0 0"/>
@@ -1499,4 +1498,5 @@
     </collision>
   </link>
+  <link name="2f_tool0"/>
   <joint name="left_finger_joint" type="revolute">
     <origin rpy="0 0 3.141592653589793" xyz="0 -0.0306011 0.054904"/>
@@ -1506,9 +1506,10 @@
     <limit effort="1000" lower="0" upper="0.8" velocity="2.0"/>
   </joint>
-  <joint name="left_left_outer_finger_joint" type="fixed">
+  <joint name="left_left_outer_finger_joint" type="fixed"> <!-- Changes type from fixed to revolute-->
     <origin rpy="0 0 0" xyz="0 0.0315 -0.0041"/>
     <parent link="left_left_outer_knuckle"/>
     <child link="left_left_outer_finger"/>
     <axis xyz="1 0 0"/>
+    <!-- <limit effort="1000" lower="0" upper="0.81" velocity="2.0"/> -->
   </joint>
   <joint name="left_left_inner_knuckle_joint" type="revolute">
@@ -1543,9 +1544,10 @@
     <mimic joint="left_finger_joint" multiplier="1" offset="0"/>
   </joint>
-  <joint name="left_right_outer_finger_joint" type="fixed">
+  <joint name="left_right_outer_finger_joint" type="fixed"> <!-- Changes type from fixed to revolute-->
     <origin rpy="0 0 0" xyz="0 0.0315 -0.0041"/>
     <parent link="left_right_outer_knuckle"/>
     <child link="left_right_outer_finger"/>
     <axis xyz="1 0 0"/>
+    <!--<limit effort="1000" lower="0" upper="0.81" velocity="2.0"/> -->
   </joint>
   <joint name="left_right_inner_knuckle_joint" type="revolute">

Commit message: 3f gripper open permanently

File: p5_ws/src/lbr_fri/lbr_fri_ros2_stack/lbr_description/urdf/dual_arm/dual_arm.xacro (robot description, xacro)
@@ -952,5 +952,5 @@
     <child link="3f_finger_1_link_1"/>
     <axis xyz="0 0 1"/>
-    <origin rpy="0 0 0" xyz="0.020 0 0"/>
+    <origin rpy="0 0 -0.43" xyz="0.020 0 0"/>
     <limit effort="100" lower="0.0495" upper="1.2218" velocity="1.23"/>
     <dynamics damping="1" friction="0.1"/>
@@ -1068,5 +1068,5 @@
     <child link="3f_finger_2_link_1"/>
     <axis xyz="0 0 1"/>
-    <origin rpy="0 0 0" xyz="0.020 0 0"/>
+    <origin rpy="0 0 -0.43" xyz="0.020 0 0"/>
     <limit effort="100" lower="0.0495" upper="1.2218" velocity="1.23"/>
     <dynamics damping="1" friction="0.1"/>
@@ -1184,5 +1184,5 @@
     <child link="3f_finger_middle_link_1"/>
     <axis xyz="0 0 1"/>
-    <origin rpy="0 0 0" xyz="0.020 0 0"/>
+    <origin rpy="0 0 -0.43" xyz="0.020 0 0"/>
     <limit effort="100" lower="0.0495" upper="1.2218" velocity="1.23"/>
     <dynamics damping="1" friction="0.1"/>

Commit message: Many different changes have been made to janise and other configurations.

File: p5_ws/src/lbr_fri/lbr_fri_ros2_stack/lbr_description/urdf/dual_arm/dual_arm.xacro (robot description, xacro)
@@ -242,5 +242,5 @@
     <child link="right_link_1"/>
     <axis xyz="0.0 0.0 1.0"/>
-    <limit effort="200" lower="-2.9670597283903604" upper="2.9670597283903604" velocity="1.710422666954443"/>
+    <limit effort="200" lower="-2.9" upper="2.9" velocity="1.710422666954443"/>
     <dynamics damping="10.0" friction="0.1"/>
   </joint>
@@ -269,5 +269,5 @@
     <child link="right_link_2"/>
     <axis xyz="0.0 1.0 0.0"/>
-    <limit effort="200" lower="-2.0943951023931953" upper="2.0943951023931953" velocity="1.710422666954443"/>
+    <limit effort="200" lower="-2" upper="2" velocity="1.710422666954443"/>
     <dynamics damping="10.0" friction="0.1"/>
   </joint>
@@ -296,5 +296,5 @@
     <child link="right_link_3"/>
     <axis xyz="0.0 0.0 1.0"/>
-    <limit effort="200" lower="-2.9670597283903604" upper="2.9670597283903604" velocity="1.7453292519943295"/>
+    <limit effort="200" lower="-2.9" upper="2.9" velocity="1.7453292519943295"/>
     <dynamics damping="10.0" friction="0.1"/>
   </joint>
@@ -323,5 +323,5 @@
     <child link="right_link_4"/>
     <axis xyz="0.0 -1.0 0.0"/>
-    <limit effort="200" lower="-2.0943951023931953" upper="2.0943951023931953" velocity="2.2689280275926285"/>
+    <limit effort="200" lower="-2" upper="2" velocity="2.2689280275926285"/>
     <dynamics damping="10.0" friction="0.1"/>
   </joint>
@@ -350,5 +350,5 @@
     <child link="right_link_5"/>
     <axis xyz="0.0 0.0 1.0"/>
-    <limit effort="200" lower="-2.9670597283903604" upper="2.9670597283903604" velocity="2.443460952792061"/>
+    <limit effort="200" lower="-2.9" upper="2.9" velocity="2.443460952792061"/>
     <dynamics damping="10.0" friction="0.1"/>
   </joint>
@@ -377,5 +377,5 @@
     <child link="right_link_6"/>
     <axis xyz="0.0 1.0 0.0"/>
-    <limit effort="200" lower="-2.0943951023931953" upper="2.0943951023931953" velocity="3.141592653589793"/>
+    <limit effort="200" lower="-2" upper="2" velocity="3.141592653589793"/>
     <dynamics damping="10.0" friction="0.1"/>
   </joint>
@@ -404,5 +404,5 @@
     <child link="right_link_7"/>
     <axis xyz="0.0 0.0 1.0"/>
-    <limit effort="200" lower="-3.0543261909900763" upper="3.0543261909900763" velocity="3.141592653589793"/>
+    <limit effort="200" lower="-3" upper="3" velocity="3.141592653589793"/>
     <dynamics damping="10.0" friction="0.1"/>
   </joint>
@@ -666,5 +666,5 @@
     <child link="left_link_1"/>
     <axis xyz="0.0 0.0 1.0"/>
-    <limit effort="200" lower="-2.9670597283903604" upper="2.9670597283903604" velocity="1.710422666954443"/>
+    <limit effort="200" lower="-2.9" upper="2.9" velocity="1.710422666954443"/>
     <dynamics damping="10.0" friction="0.1"/>
   </joint>
@@ -693,5 +693,5 @@
     <child link="left_link_2"/>
     <axis xyz="0.0 1.0 0.0"/>
-    <limit effort="200" lower="-2.0943951023931953" upper="2.0943951023931953" velocity="1.710422666954443"/>
+    <limit effort="200" lower="-2" upper="2" velocity="1.710422666954443"/>
     <dynamics damping="10.0" friction="0.1"/>
   </joint>
@@ -720,5 +720,5 @@
     <child link="left_link_3"/>
     <axis xyz="0.0 0.0 1.0"/>
-    <limit effort="200" lower="-2.9670597283903604" upper="2.9670597283903604" velocity="1.7453292519943295"/>
+    <limit effort="200" lower="-2.9" upper="2.9" velocity="1.7453292519943295"/>
     <dynamics damping="10.0" friction="0.1"/>
   </joint>
@@ -747,5 +747,5 @@
     <child link="left_link_4"/>
     <axis xyz="0.0 -1.0 0.0"/>
-    <limit effort="200" lower="-2.0943951023931953" upper="2.0943951023931953" velocity="2.2689280275926285"/>
+    <limit effort="200" lower="-2" upper="2" velocity="2.2689280275926285"/>
     <dynamics damping="10.0" friction="0.1"/>
   </joint>
@@ -774,5 +774,5 @@
     <child link="left_link_5"/>
     <axis xyz="0.0 0.0 1.0"/>
-    <limit effort="200" lower="-2.9670597283903604" upper="2.9670597283903604" velocity="2.443460952792061"/>
+    <limit effort="200" lower="-2.9" upper="2.9" velocity="2.443460952792061"/>
     <dynamics damping="10.0" friction="0.1"/>
   </joint>
@@ -801,5 +801,5 @@
     <child link="left_link_6"/>
     <axis xyz="0.0 1.0 0.0"/>
-    <limit effort="200" lower="-2.0943951023931953" upper="2.0943951023931953" velocity="3.141592653589793"/>
+    <limit effort="200" lower="-2" upper="2" velocity="3.141592653589793"/>
     <dynamics damping="10.0" friction="0.1"/>
   </joint>
@@ -828,5 +828,5 @@
     <child link="left_link_7"/>
     <axis xyz="0.0 0.0 1.0"/>
-    <limit effort="200" lower="-3.0543261909900763" upper="3.0543261909900763" velocity="3.141592653589793"/>
+    <limit effort="200" lower="-3" upper="3" velocity="3.141592653589793"/>
     <dynamics damping="10.0" friction="0.1"/>
   </joint>

Commit message: Fixed URDF point

File: p5_ws/src/lbr_fri/lbr_fri_ros2_stack/lbr_description/urdf/dual_arm/dual_arm.xacro (robot description, xacro)
@@ -1701,5 +1701,5 @@
     <parent link="left_link_ee"/>
     <child link="2f_tool0"/>
-    <origin rpy="0 3.14 0" xyz="0 0 0.175"/>
+    <origin rpy="0 3.14 0" xyz="0 0 0.165"/>
   </joint>
 </robot>
